Commit message: added realsense TF

File: urdf/driller.urdf (robot description, URDF)
Before this commit: robot driller, 15 links, 14 joints
Links:
- added link camera_link
- added link robot_chassis, mass 3; collision box size=1.5 3 0.5; visual mesh filename=package://robot_model/meshes/base_link.dae
- link base_link: mass 3 -> None; geometry 
Joints:
- added joint base_link_to_chassis: type fixed, parent base_link, child robot_chassis
- added joint robot_to_camera: type fixed, parent base_link, child camera_link, origin xyz=0 -1.2 0.8 rpy=0 0 -1.57075
- joint base_to_left_lower_arm: parent base_link -> robot_chassis
- joint base_to_left_lower_leg: parent base_link -> robot_chassis
- joint base_to_left_upper_arm: parent base_link -> robot_chassis
- joint base_to_left_upper_leg: parent base_link -> robot_chassis
- joint base_to_left_wheel_leg: parent base_link -> robot_chassis
- joint base_to_left_wheel_steering: parent base_link -> robot_chassis
- joint base_to_right_lower_arm: parent base_link -> robot_chassis
- joint base_to_right_lower_leg: parent base_link -> robot_chassis
- joint base_to_right_upper_arm: parent base_link -> robot_chassis
- joint base_to_right_upper_leg: parent base_link -> robot_chassis
- joint base_to_right_wheel_leg: parent base_link -> robot_chassis
- joint base_to_right_wheel_steering: parent base_link -> robot_chassis

Commit message: Added support for open source tracking

File: urdf/driller.urdf (robot description, URDF)
Before this commit: robot driller, 17 links, 16 joints
Links:
- added link map
- added link odom
- link left_lower_arm: geometry visual mesh filename=package://robot_model/meshes/wheel_arm.dae scale=0.1 0.1 0.1
- link left_lower_leg: geometry visual mesh filename=package://robot_model/meshes/wheel_arm.dae scale=0.1 0.1 0.1
- link left_upper_arm: geometry visual mesh filename=package://robot_model/meshes/wheel_arm.dae scale=0.1 0.1 0.1
- link left_upper_leg: geometry visual mesh filename=package://robot_model/meshes/wheel_arm.dae scale=0.1 0.1 0.1
- link left_wheel_arm: geometry collision cylinder length=0.022 radius=0.035; visual mesh filename=package://robot_model/meshes/wheel.dae scale=0.1 0.1 0.1
- link left_wheel_leg: geometry collision cylinder length=0.022 radius=0.035; visual mesh filename=package://robot_model/meshes/wheel.dae scale=0.1 0.1 0.1
- link left_wheel_steering: geometry visual mesh filename=package://robot_model/meshes/front_steer.dae scale=0.1 0.1 0.1
- link right_lower_arm: geometry visual mesh filename=package://robot_model/meshes/wheel_arm.dae scale=0.1 0.1 0.1
- link right_lower_leg: geometry visual mesh filename=package://robot_model/meshes/wheel_arm.dae scale=0.1 0.1 0.1
- link right_upper_arm: geometry visual mesh filename=package://robot_model/meshes/wheel_arm.dae scale=0.1 0.1 0.1
- link right_upper_leg: geometry visual mesh filename=package://robot_model/meshes/wheel_arm.dae scale=0.1 0.1 0.1
- link right_wheel_arm: geometry collision cylinder length=0.022 radius=0.035; visual mesh filename=package://robot_model/meshes/wheel.dae scale=0.1 0.1 0.1
- link right_wheel_leg: geometry collision cylinder length=0.022 radius=0.035; visual mesh filename=package://robot_model/meshes/wheel.dae scale=0.1 0.1 0.1
- link right_wheel_steering: geometry visual mesh filename=package://robot_model/meshes/front_steer.dae scale=0.1 0.1 0.1
- link robot_chassis: geometry collision box size=0.15 0.3 0.05; visual mesh filename=package://robot_model/meshes/base_link.dae scale=0.1 0.1 0.1
Joints:
- removed joint robot_to_camera
- added joint camera_to_robot: type fixed, parent camera_link, child base_link, origin xyz=-0.12 0 -0.08 rpy=0 0 1.57075
- added joint map_to_odom: type fixed, parent map, child odom
- added joint odom_to_camera_link: type fixed, parent odom, child camera_link
- joint base_to_left_lower_arm: origin xyz=0.29 -0.95 0.1 -> xyz=0.029 -0.095 0.01
- joint base_to_left_lower_leg: origin xyz=0.29 1.52 0.1 -> xyz=0.029 0.152 0.01
- joint base_to_left_upper_arm: origin xyz=0.29 -0.95 0.42 -> xyz=0.029 -0.095 0.042
- joint base_to_left_upper_leg: origin xyz=0.29 1.52 0.42 -> xyz=0.029 0.152 0.042
- joint base_to_left_wheel_arm: origin xyz=0.05 0 0 -> xyz=0.005 0 0
- joint base_to_left_wheel_leg: origin xyz=0.9 1.52 0.05 -> xyz=0.09 0.152 0.005
- joint base_to_left_wheel_steering: origin xyz=0.85 -0.95 0.05 -> xyz=0.085 -0.095 0.005
- joint base_to_right_lower_arm: origin xyz=-0.29 -0.95 0.1 -> xyz=-0.029 -0.095 0.01
- joint base_to_right_lower_leg: origin xyz=-0.29 1.52 0.1 -> xyz=-0.029 0.152 0.01
- joint base_to_right_upper_arm: origin xyz=-0.29 -0.95 0.42 -> xyz=-0.029 -0.095 0.042
- joint base_to_right_upper_leg: origin xyz=-0.29 1.52 0.42 -> xyz=-0.029 0.152 0.042
- joint base_to_right_wheel_arm: origin xyz=-0.05 0 0 -> xyz=-0.005 0 0
- joint base_to_right_wheel_leg: origin xyz=-0.9 1.52 0.05 -> xyz=-0.09 0.152 0.005
- joint base_to_right_wheel_steering: origin xyz=-0.85 -0.95 0.05 -> xyz=-0.085 -0.095 0.005
